File: circuit/circuit.brd (EAGLE design)
At the start: 40.6 x 22.9 mm, 14 parts, among them J1 AVR_SPI_PRG_6PTH

Commit message: update
Parts:
- moved JP2 12.7 mm to (38.1, 17.8)
Routing:
- net GND: track 91.6 -> 83.0 mm
- net VBUS: track 59.2 -> 59.8 mm
Changed lines of the file:
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@@
 <element name="R9" library="my" package="1/4W-5.08V" value="6.8k" x="12.7" y="10.16" rot="R180"/>
 <element name="U$2" library="avr-7" package="DIL08" value="TINY13A" x="19.05" y="11.43" rot="R90"/>
-<element name="JP2" library="SparkFun-Connectors" package="1X02" value="" x="38.1" y="5.08" rot="R90"/>
+<element name="JP2" library="SparkFun-Connectors" package="1X02" value="" x="38.1" y="17.78" rot="R90"/>
 <element name="U$1" library="my" package="TO-92" value="S-812C33AY-B-G" x="30.48" y="17.78" rot="R270"/>
 <element name="JP3" library="SparkFun-Connectors" package="1X03" value="" x="25.4" y="10.16" rot="R90"/>
@@
 <contactref element="U$1" pad="1"/>
 <wire x1="22.86" y1="20.32" x2="38.1" y2="20.32" width="1.27" layer="16"/>
-<wire x1="38.1" y1="20.32" x2="38.1" y2="11.43" width="1.27" layer="16"/>
-<wire x1="38.1" y1="11.43" x2="38.1" y2="7.62" width="1.27" layer="16"/>
 <wire x1="22.86" y1="15.24" x2="22.86" y2="20.32" width="0.6096" layer="16"/>
 <wire x1="27.94" y1="5.08" x2="29.21" y2="5.08" width="0.3048" layer="1"/>
-<wire x1="29.21" y1="5.08" x2="29.21" y2="11.43" width="0.3048" layer="1"/>
-<wire x1="29.21" y1="11.43" x2="38.1" y2="11.43" width="0.3048" layer="1"/>
-<via x="38.1" y="11.43" extent="1-16" drill="0.6" shape="square"/>
+<wire x1="29.21" y1="5.08" x2="29.21" y2="12.7" width="0.3048" layer="1"/>
+<wire x1="29.21" y1="12.7" x2="38.1" y2="20.32" width="0.3048" layer="1"/>
+<via x="38.1" y="20.32" extent="1-16" drill="0.6" shape="square"/>
 <contactref element="JP3" pad="3"/>
 <wire x1="25.4" y1="15.24" x2="22.86" y2="15.24" width="0.4064" layer="16"/>
@@
 <wire x1="4.94" y1="7.93" x2="4.94" y2="5.22" width="1.27" layer="16"/>
 <wire x1="4.94" y1="5.22" x2="7.62" y2="2.54" width="1.27" layer="16"/>
-<wire x1="7.62" y1="2.54" x2="36.195" y2="2.54" width="1.27" layer="16"/>
-<wire x1="36.195" y1="2.54" x2="38.1" y2="5.08" width="1.27" layer="16"/>
+<wire x1="7.62" y1="2.54" x2="38.1" y2="2.54" width="1.27" layer="16"/>
+<wire x1="38.1" y1="2.54" x2="38.1" y2="17.78" width="1.27" layer="16"/>
 <contactref element="U$1" pad="2"/>
 <wire x1="30.48" y1="17.78" x2="33.02" y2="17.78" width="0.6096" layer="16"/>
-<wire x1="33.02" y1="17.78" x2="36.195" y2="17.78" width="0.6096" layer="16"/>
-<wire x1="36.195" y1="17.78" x2="36.195" y2="2.54" width="0.6096" layer="16"/>
+<wire x1="33.02" y1="17.78" x2="38.1" y2="17.78" width="0.6096" layer="16"/>
 </signal>
 <signal name="3.3V">
